Commit message: added chess-playing dobot robot sim with vision, motion and lobotlab backend

File: sim/urdf/dobot_magician.urdf (robot description, URDF)
Before this commit: robot dobot_magician, 5 links, 4 joints
Links:
- added link jaw_left, mass 0.02; collision box size=0.02 0.005 0.014; visual box size=0.02 0.005 0.014
- added link jaw_right, mass 0.02; collision box size=0.02 0.005 0.014; visual box size=0.02 0.005 0.014
- link tool: geometry collision cylinder length=0.024 radius=0.010; visual cylinder length=0.04 radius=0.012
Joints:
- added joint joint_gripper_l: type prismatic, parent tool, child jaw_left, origin xyz=0.04 -0.0025 0 rpy=0 0 0, axis 0 1 0, limit lower=-0.0135 upper=0 effort=20 velocity=0.5
- added joint joint_gripper_r: type prismatic, parent tool, child jaw_right, origin xyz=0.04 0.0025 0 rpy=0 0 0, axis 0 1 0, limit lower=0 upper=0.0135 effort=20 velocity=0.5
- joint joint4: axis (none) -> 0 1 0; limit (none) -> lower=-2.618 upper=2.618 effort=20 velocity=1.0; type fixed -> revolute

File: sim/urdf/dobot_magician_ros.urdf (robot description, URDF)
Before this commit: robot magician, 10 links, 9 joints
Joints:
- joint magician_joint_mimic_1: limit lower=0.0 upper=6.283185307179586 effort=2000 velocity=1 -> lower=-7.0 upper=7.0 effort=2000 velocity=1
- joint magician_joint_mimic_2: limit lower=0.0 upper=6.283185307179586 effort=2000 velocity=1 -> lower=-7.0 upper=7.0 effort=2000 velocity=1
